Commit message: Added Nav Stack

File: ugv_sim/scout/scout_description/urdf/scout_v2.xacro (robot description, xacro)
@@ -18,5 +18,5 @@
     <xacro:property name="wheel_radius" value="1.6459e-01" />
     <!-- Base link -->
-    <link name="base_link">
+    <link name="scout_base_link">
         <visual>
             <origin xyz="0 0 0" rpy="0 0 0" />
@@ -43,5 +43,5 @@
         <child link="chassis_link" />
     </joint> -->
-    <link name="inertial_link">
+    <link name="scout_inertial_link">
         <inertial>
             <mass value="50" />
@@ -53,8 +53,8 @@
         </inertial>
     </link>
-    <joint name="inertial_joint" type="fixed">
+    <joint name="scout_inertial_joint" type="fixed">
         <origin xyz="0 0 0" rpy="0 0 0" />
-        <parent link="base_link" />
-        <child link="inertial_link" />
+        <parent link="scout_base_link" />
+        <child link="scout_inertial_link" />
     </joint>
     <!-- For testing, hang the robot up in the air -->

File: ugv_sim/scout/scout_description/urdf/scout_v2_ur3e.xacro (robot description, xacro)
@@ -17,9 +17,5 @@
     <xacro:property name="wheel_length" value="1.1653e-01" />
     <xacro:property name="wheel_radius" value="1.6459e-01" />
-    <!-- Base link -->
-    <!-- <xacro:include filename="$(find scout_description)/urdf/scout_v2.xacro"/> -->
-    <!-- <xacro:scout_v2 wheel_prefix="front_left">
-        <origin xyz="${wheelbase/2} ${track/2} ${wheel_vertical_offset}" rpy="0 0 0" />
-    </xacro:scout_wheel_type2> -->
+    <!-- SCOUT -->
     <link name="scout_base_link">
         <visual>
@@ -47,5 +43,5 @@
         <child link="chassis_link" />
     </joint> -->
-    <link name="inertial_link">
+    <link name="scout_inertial_link">
         <inertial>
             <mass value="50" />
@@ -57,13 +53,6 @@
         <origin xyz="0 0 0" rpy="0 0 0" />
         <parent link="scout_base_link" />
-        <child link="inertial_link" />
+        <child link="scout_inertial_link" />
     </joint>
-    <!-- For testing, hang the robot up in the air -->
-    <!-- <link name="world" />
-    <joint name="world_to_base_link=" type="fixed">
-        <origin xyz="0 0 0.5" rpy="0 0 0" />
-        <parent link="world"/>
-        <child link="base_link"/>
-    </joint> -->
     <!-- Scout wheel macros -->
     <!-- wheel labeled from 0 to 3, conter-clockwise, starting from front right wheel -->
@@ -82,12 +71,4 @@
     </xacro:scout_wheel_type2>
     <!-- UR3E Insert -->
-    <!-- Instantiate the Gazebo robot and pass it all the required arguments. -->
-    <!-- <xacro:include filename="$(find ur_description)/urdf/inc/ur3e_macro.xacro"/>
-    <xacro:ur3e_robot
-      prefix="ur3e"
-      originx="${-base_y_size+0.1}"
-      originy="0"
-      originz="${0.5 * 0.152}"
-      /> -->
     <!--Parameter files -->
     <xacro:arg name="joint_limit_params" default="$(find ur_description)/config/ur3e/joint_limits.yaml"/>
@@ -100,18 +81,4 @@
     <xacro:arg name="safety_pos_margin" default="0.15" doc="The lower/upper limits in the safety controller" />
     <xacro:arg name="safety_k_position" default="20" doc="Used to set k position in the safety controller" />
-    <!-- <xacro:arg name="robot_model" default="ur3e" /> -->
-<!--
-    <xacro:include filename="$(find ur_gazebo)/urdf/ur_macro.xacro"/>
-    <xacro:ur_robot_gazebo
-      prefix=""
-      joint_limits_parameters_file="$(arg joint_limit_params)"
-      kinematics_parameters_file="$(arg kinematics_params)"
-      physical_parameters_file="$(arg physical_params)"
-      visual_parameters_file="$(arg visual_params)"
-      transmission_hw_interface="$(arg transmission_hw_interface)"
-      safety_limits="$(arg safety_limits)"
-      safety_pos_margin="$(arg safety_pos_margin)"
-      safety_k_position="$(arg safety_k_position)"
-      /> -->
     <xacro:include filename="$(find ur_description)/urdf/inc/ur_macro.xacro"/>
     <xacro:ur_robot
@@ -132,43 +99,84 @@
       <origin xyz="${base_y_size-0.1} 0 ${base_z_size-0.09}" rpy="0 0 ${pi}"/>
     </joint>
-    <!--Cylinder insert-->
-    <!-- <xacro:property name="r" value="0.02" />
-    <xacro:property name="h" value="0.25" /> -->
-    <!-- <link name="cylinder_link">
-    <visual>
-      <origin xyz="${base_y_size-0.1} ${0} ${base_z_size}" rpy="0 0 0"/>
-      <geometry>
-        <cylinder length="${h}" radius="${r}"/>
-      </geometry>
-      <material name="green">
-        <color rgba="0 1 0 1"/>
-      </material>
-    </visual>
-    <inertial>
-      <origin xyz="0 0 0" rpy="0 0 0"/>
-      <mass value="0.05"/>
-      <inertia ixx="0.001"  ixy="0"  ixz="0" iyy="0.001" iyz="0" izz="0.001" />
-    </inertial>
-    <collision>
-      <origin xyz="0 0 0" rpy="0 0 0"/>
-      <geometry>
-        <cylinder length="${h}" radius="${r}"/>
-      </geometry>
-    </collision>
-  </link> -->
-  <!-- <gazebo reference="cylinder_link">
-    <material>Gazebo/Grey</material>
-    <dampingFactor>0.005</dampingFactor>
-    <kp>1000000</kp>
-    <kd>1.0</kd>
-    <mu1>100.0</mu1>
-    <mu2>100.0</mu2>
-    <minDepth>0.001</minDepth>
-  </gazebo>
-  <joint name="cylinder_joint" type="fixed">
-      <parent link="base_link"/>
-      <child link="cylinder_link"/>
-      <axis xyz="0 0 0" rpy="0 0 0" />
-  </joint> -->
+    <!-- LIDAR -->
+    <!-- <xacro:property name="M_PI" value="3.1415926535897931" />
+    <xacro:include filename="$(find velodyne_description)/urdf/VLP-16.urdf.xacro"/>
+    <xacro:VLP-16 parent="scout_base_link" name="velodyne"
+        topic="/velodyne_points" hz="10" gpu="false"
+        organize_cloud="false" lasers:="16" samples="1875" collision_range="0.3"
+        min_range="0.9" max_range="130.0" noise="0.0" min_angle="-${M_PI}" max_angle="${M_PI}">
+        <origin xyz="0 0 0.4" rpy="0 0 0" />
+    </xacro:VLP-16> -->
+    <link name="laser_frame">
+      <inertial>
+        <mass value="0.425"/>
+        <origin xyz="0 0 0.003675" rpy="0 0 0" />
+        <inertia ixx="0.000308429" ixy="0" ixz="0"
+                  iyy="0.000308429" iyz="0" izz="0.00034589"/>
+      </inertial>
+      <collision name="lidar_collision">
+        <origin xyz="0 0 0.03675" rpy="0 0 0" />
+        <geometry>
+          <cylinder radius="0.04350" length="0.07350"/>
+        </geometry>
+      </collision>
+      <visual name="lidar_visual">
+        <origin xyz="0 0 0.0" rpy="0 0 0"/>
+        <geometry>
+          <mesh filename="$(find scout_description)/meshes/os1_64.stl" />
+        </geometry>
+      </visual>
+    </link>
+    <joint name="laser_joint" type="fixed">
+      <parent link="scout_base_link"/>
+      <child link="laser_frame"/>
+      <origin xyz="${base_y_size+0.05} 0 ${0.0}" rpy="0 0 0"/>
+    </joint>
+    <!-- Add lidar plugin for scan topic -->
+    <gazebo reference="laser_frame">
+        <material>Gazebo/Red</material>
+        <sensor name="laser" type="ray">
+            <pose> 0 0 0 0 0 0 </pose>
+            <visualize>true</visualize>
+            <update_rate>10</update_rate>
+            <ray>
+                <scan>
+                    <horizontal>
+                        <resolution>1</resolution>
+                        <samples>180</samples>
+                        <min_angle>-1.57</min_angle>
+                        <max_angle>1.57</max_angle>
+                    </horizontal>
+                </scan>
+                <range>
+                    <resolution>0.1</resolution>
+                    <min>0.3</min>
+                    <max>100</max>
+                </range>
+            </ray>
+            <plugin name="laser_controller" filename="libgazebo_ros_laser.so">
+                <topicName>/scan</topicName>
+                <frameName>laser_frame</frameName>
+            </plugin>
+        </sensor>
+    </gazebo>
+    <!-- Add Skid steer controller for odom topic -->
+    <gazebo>
+        <plugin name="skid_steer_drive_controller" filename="libgazebo_ros_skid_steer_drive.so">
+            <updateRate>100.0</updateRate>
+            <robotNamespace>/</robotNamespace>
+            <leftFrontJoint>front_left_wheel</leftFrontJoint>
+            <rightFrontJoint>front_right_wheel</rightFrontJoint>
+            <leftRearJoint>rear_left_wheel</leftRearJoint>
+            <rightRearJoint>rear_right_wheel</rightRearJoint>
+            <wheelSeparation>4</wheelSeparation>
+            <robotBaseFrame>scout_base_link</robotBaseFrame>
+            <commandTopic>cmd_vel</commandTopic>
+            <broadcastTF>true</broadcastTF>
+            <odometrySource>world</odometrySource>
+            <odometryTopic>odom</odometryTopic>
+            <odometryFrame>odom</odometryFrame>
+        </plugin>
+    </gazebo>
     <!-- Additional definitions -->
     <xacro:include filename="$(arg urdf_extras)" />
