Commit message: Fixed scout + ur3e bugs and added ik script

File: ugv_sim/scout/scout_description/urdf/scout_v2_ur3e.xacro (robot description, xacro)
@@ -6,5 +6,4 @@
     <xacro:include filename="$(find scout_description)/urdf/scout_wheel_type1.xacro" />
     <xacro:include filename="$(find scout_description)/urdf/scout_wheel_type2.xacro" />
-    <!-- <xacro:include filename"$(find scout_description)/urdf/cylinder.xacro" /> -->
     <!-- Variables -->
     <xacro:property name="M_PI" value="3.14159"/>
@@ -19,4 +18,8 @@
     <xacro:property name="wheel_radius" value="1.6459e-01" />
     <!-- Base link -->
+    <!-- <xacro:include filename="$(find scout_description)/urdf/scout_v2.xacro"/> -->
+    <!-- <xacro:scout_v2 wheel_prefix="front_left">
+        <origin xyz="${wheelbase/2} ${track/2} ${wheel_vertical_offset}" rpy="0 0 0" />
+    </xacro:scout_wheel_type2> -->
     <link name="scout_base_link">
         <visual>
@@ -47,7 +50,4 @@
         <inertial>
             <mass value="50" />
-            <!-- <mass value="50" /> -->
-            <!-- <origin xyz="-0.00065 -0.085 0.062" />
-            <inertia ixx="0.6022" ixy="-0.02364" ixz="-0.1197" iyy="1.7386" iyz="-0.001544" izz="2.0296" /> -->
             <origin xyz="0.0 0.0 0.0" />
             <inertia ixx="2.288641" ixy="0" ixz="0" iyy="5.103976" iyz="0" izz="3.431465" />
@@ -112,7 +112,4 @@
       safety_pos_margin="$(arg safety_pos_margin)"
       safety_k_position="$(arg safety_k_position)"
-      originx="${-base_y_size+0.1}"
-      originy="0"
-      originz="${base_z_size}"
       /> -->
     <xacro:include filename="$(find ur_description)/urdf/inc/ur_macro.xacro"/>

Commit message: fixed lidar collision

File: ugv_sim/scout/scout_description/urdf/scout_v2_ur3e.xacro (robot description, xacro)
@@ -99,4 +99,25 @@
       <origin xyz="${base_y_size-0.1} 0 ${base_z_size-0.09}" rpy="0 0 ${pi}"/>
     </joint>
+    <!-- Drilling end effector -->
+    <!-- <link name="drill_end_effector_link">
+        <visual>
+            <geometry>
+                <mesh filename="package://scout_description/meshes/poly_drill/drilling_end_effector.dae" />
+            </geometry>
+            <origin xyz="0 0 0" rpy="0 0 0" />
+        </visual>
+        <collision>
+            <geometry>
+                <mesh filename="package://scout_description/meshes/poly_drill/drilling_end_effector.dae" />
+            </geometry>
+            <origin xyz="0 0 0" rpy="0 0 0" />
+        </collision>
+    </link>
+    <joint name="drill_end_effector_joint" type="fixed">
+      <parent link="wrist_3_link"/>
+      <child link="drill_end_effector_link"/>
+      <axis xyz="0 0 0" rpy="0 0 0" />
+      <origin xyz="0 0 0.005" rpy="${pi} 0 0"/>
+    </joint> -->
     <!-- LIDAR -->
     <!-- <xacro:property name="M_PI" value="3.1415926535897931" />
@@ -116,8 +137,8 @@
       </inertial>
       <collision name="lidar_collision">
-        <origin xyz="0 0 0.03675" rpy="0 0 0" />
-        <geometry>
-          <cylinder radius="0.04350" length="0.07350"/>
-        </geometry>
+        <!-- <origin xyz="0 0 0.03675" rpy="0 0 0" /> -->
+        <!-- <geometry> -->
+          <!-- <cylinder radius="0.04350" length="0.07350"/> -->
+        <!-- </geometry> -->
       </collision>
       <visual name="lidar_visual">
@@ -131,5 +152,5 @@
       <parent link="scout_base_link"/>
       <child link="laser_frame"/>
-      <origin xyz="${base_y_size+0.05} 0 ${0.0}" rpy="0 0 0"/>
+      <origin xyz="${base_y_size+0.02} 0 ${0.0}" rpy="0 0 0"/>
     </joint>
     <!-- Add lidar plugin for scan topic -->

Commit message: fixed manipulation reference frame

File: ugv_sim/scout/scout_description/urdf/scout_v2_ur3e.xacro (robot description, xacro)
@@ -136,10 +136,10 @@
                   iyy="0.000308429" iyz="0" izz="0.00034589"/>
       </inertial>
-      <collision name="lidar_collision">
-        <!-- <origin xyz="0 0 0.03675" rpy="0 0 0" /> -->
-        <!-- <geometry> -->
-          <!-- <cylinder radius="0.04350" length="0.07350"/> -->
-        <!-- </geometry> -->
-      </collision>
+      <!-- <collision name="lidar_collision">
+        <origin xyz="0 0 0.03675" rpy="0 0 0" />
+        <geometry>
+          <cylinder radius="0.04350" length="0.07350"/>
+        </geometry>
+      </collision> -->
       <visual name="lidar_visual">
         <origin xyz="0 0 0.0" rpy="0 0 0"/>
@@ -152,5 +152,5 @@
       <parent link="scout_base_link"/>
       <child link="laser_frame"/>
-      <origin xyz="${base_y_size+0.02} 0 ${0.0}" rpy="0 0 0"/>
+      <origin xyz="${base_y_size+0.02} 0 ${0.1}" rpy="0 0 0"/>
     </joint>
     <!-- Add lidar plugin for scan topic -->
@@ -182,4 +182,18 @@
         </sensor>
     </gazebo>
+    <!-- NOT WORKING: Gazebo ODOM plugin -->
+    <!-- <gazebo>
+        <plugin name="p3e_odometry" filename="libgazebo_ros_p3d.so">
+            <frameName>map</frameName>
+            <alwaysOn>true</alwaysOn>
+            <robotNamespace></robotNamespace>
+            <bodyName>scout_base_link</bodyName>
+            <topicName>odom</topicName>
+            <updateRate>100.0</updateRate>
+            <gaussianNoise>0.0</gaussianNoise>
+            <xyzOffsets>0 0 0</xyzOffsets>
+            <rpyOffsets>0 0 0</rpyOffsets>
+        </plugin>
+    </gazebo> -->
     <!-- Add Skid steer controller for odom topic -->
     <gazebo>
@@ -195,7 +209,10 @@
             <commandTopic>cmd_vel</commandTopic>
             <broadcastTF>true</broadcastTF>
-            <odometrySource>world</odometrySource>
+            <!-- <odometrySource>map</odometrySource> -->
             <odometryTopic>odom</odometryTopic>
             <odometryFrame>odom</odometryFrame>
+            <covariance_x>0.0</covariance_x>
+            <covariance_y>0.0</covariance_y>
+            <covariance_yaw>0.0</covariance_yaw>
         </plugin>
     </gazebo>
